File: schematics/backplane/backplane/leds.kicad_sch (KiCad schematic)
At the start: 31 parts, among them J13 MCP rest pins, Q11 NX138BKMYL, Q12 NX138BKMYL, Q13 NX138BKMYL, U5 MCP23017_SO, U6 74HC14

Commit message: Add crystal data and Test points
Other:
- title: (none) -> Status LEDs
Changed lines of the file:
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@@
 	(generator_version "8.0")
 	(paper "A4")
+	(title_block
+		(title "Status LEDs")
+	)
 	(junction
 		(at 72.39 105.41)

Commit message: redo numbering
Parts:
- renumbered C31 to C32, C32 to C33, D6 to D1, D7 to D2, D8 to D3, D9 to D4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
